File: Eagle/k1fm-pico-balloon-v1.3.brd (EAGLE design)
At the start: 26.7 x 41.1 mm, 40 parts, among them J1 I2C, J2 ICSP, J3 SERIAL, J4 POWER, Q1 ASTX-H11-25.000MHZ-T, Q2 DMP2305U, Q3 DMP2305U, U1 ATMEGA328, U2 Si5351A-B-GT, U3 MCP1754X-XXXXX/C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

Commit message: Remove wire stubs
Routing:
- net 3V: track 106.5 -> 105.1 mm
Changed lines of the file:
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@@
 <via x="14.3971125" y="74.66815" extent="1-16" drill="0.2"/>
 <via x="13.348934375" y="69.3406125" extent="1-16" drill="0.2"/>
-<wire x1="18.947928125" y1="70.45523125" x2="15.21810625" y2="70.45523125" width="0.1524" layer="1"/>
+<wire x1="18.947928125" y1="70.45523125" x2="15.59775625" y2="70.45523125" width="0.1524" layer="1"/>
 </signal>
 <signal name="3V">
@@
 <wire x1="14.3156125" y1="52.028271875" x2="9.806440625" y2="56.53744375" width="0.1524" layer="2"/>
 <wire x1="9.806440625" y1="56.53744375" x2="7.428621875" y2="56.53744375" width="0.1524" layer="2"/>
-<wire x1="14.843965625" y1="54.377925" x2="14.843965625" y2="54.11790625" width="0.1524" layer="1"/>
-<wire x1="14.843965625" y1="54.11790625" x2="14.1030125" y2="53.376953125" width="0.1524" layer="1"/>
 <wire x1="14.1030125" y1="53.376953125" x2="13.97363125" y2="53.376953125" width="0.1524" layer="1"/>
 <wire x1="9.07876875" y1="63.3856875" x2="8.7500375" y2="63.05695625" width="0.1524" layer="1"/>
